File: Devboard/CH552Devboard/CH552Devboard.sch (KiCad schematic (older format))
At the start: 16 parts, among them J1 D+, J2 USB_B_Micro, J3 System, J4 GPIO, SW1 SW_Push, SW2 SW_Push, SW3 SW_Push, SW4 SW_Push, U1 CH552T

Commit message: Finished and ordered PlasticFrog v1
Parts:
- U1: symbol CH552:CH552T -> CH552Devboard-rescue:CH552T-CH552
Changed lines of the file:
@@
 $EndDescr
 $Comp
-L CH552:CH552T U1
+L CH552Devboard-rescue:CH552T-CH552 U1
 U 1 1 5C6D8296
 P 6300 3450
@@
 	6850 3800 7200 3800
 $Comp
-L power:VSS #PWR?
+L power:VSS #PWR0104
 U 1 1 5C7F52C2
 P 7750 3200
-F 0 "#PWR?" H 7750 3050 50  0001 C CNN
+F 0 "#PWR0104" H 7750 3050 50  0001 C CNN
 F 1 "VSS" V 7767 3328 50  0000 L CNN
 F 2 "" H 7750 3200 50  0001 C CNN
@@
 $EndComp
 $Comp
-L power:VSS #PWR?
+L power:VSS #PWR0105
 U 1 1 5C7F52ED
 P 6950 2750
-F 0 "#PWR?" H 6950 2600 50  0001 C CNN
+F 0 "#PWR0105" H 6950 2600 50  0001 C CNN
 F 1 "VSS" V 6967 2878 50  0000 L CNN
 F 2 "" H 6950 2750 50  0001 C CNN
