File: BusinessCard/Schematics/Card.kicad_pcb (KiCad board)
At the start: 2 copper layers, 88.1 x 50.2 mm, 18 parts, among them J1 USB_A, J2 System, J3 ExpansionPort, J4 CapPad1, J5 CapPad2, J6 Programming Port, U1 CH552T

Commit message: Cleaned up card schematics
Routing:
- net VSS: track 10.3 -> 2.33 mm, vias 2 -> 0
- net VCC: track 50.2 -> 45.2 mm
- net +3V3: track 33.5 -> 31.1 mm
Changed lines of the file:
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@@
     (thickness 1.6)
     (drawings 71)
-    (tracks 78)
+    (tracks 70)
     (zones 0)
     (modules 18)
@@
   (segment (start 107.775 132.6) (end 111 129.375) (width 0.25) (layer F.Cu) (net 1))
   (segment (start 105.8 132.6) (end 107.775 132.6) (width 0.25) (layer F.Cu) (net 1))
-  (segment (start 105.8 132.925) (end 103.2 135.525) (width 0.25) (layer F.Cu) (net 1))
-  (segment (start 105.8 132.8) (end 105.8 132.925) (width 0.25) (layer F.Cu) (net 1))
-  (segment (start 103.2 150.6) (end 104 151.4) (width 0.25) (layer F.Cu) (net 1))
-  (segment (start 103.8 151.2) (end 104 151.4) (width 0.25) (layer F.Cu) (net 1))
-  (segment (start 103.2 135.525) (end 103.2 150.6) (width 0.25) (layer F.Cu) (net 1))
-  (segment (start 104 151.4) (end 108.4 155.8) (width 0.25) (layer F.Cu) (net 1))
+  (segment (start 105.8 153.2) (end 108.4 155.8) (width 0.25) (layer F.Cu) (net 1))
+  (segment (start 105.8 132.8) (end 105.8 153.2) (width 0.25) (layer F.Cu) (net 1))
   (segment (start 110.025 128.25) (end 111 128.25) (width 0.25) (layer F.Cu) (net 2))
   (segment (start 107.7 128.25) (end 110.025 128.25) (width 0.25) (layer F.Cu) (net 2))
   (segment (start 106.55 129.4) (end 107.7 128.25) (width 0.25) (layer F.Cu) (net 2))
   (segment (start 105.8 129.4) (end 106.55 129.4) (width 0.25) (layer F.Cu) (net 2))
-  (segment (start 102.593398 152.533398) (end 105.86 155.8) (width 0.25) (layer F.Cu) (net 2))
-  (segment (start 102.593398 125) (end 102.593398 152.533398) (width 0.25) (layer F.Cu) (net 2))
   (segment (start 97.896699 120.303301) (end 102.593398 125) (width 0.25) (layer F.Cu) (net 2))
   (segment (start 105.8 128.206602) (end 105.8 129.4) (width 0.25) (layer F.Cu) (net 2))
   (segment (start 102.593398 125) (end 105.8 128.206602) (width 0.25) (layer F.Cu) (net 2))
+  (segment (start 105.8 130.275) (end 105.8 129.4) (width 0.25) (layer F.Cu) (net 2))
+  (segment (start 104.974999 131.100001) (end 105.8 130.275) (width 0.25) (layer F.Cu) (net 2))
+  (segment (start 104.974999 153.712918) (end 104.974999 131.100001) (width 0.25) (layer F.Cu) (net 2))
+  (segment (start 105.86 154.597919) (end 104.974999 153.712918) (width 0.25) (layer F.Cu) (net 2))
+  (segment (start 105.86 155.8) (end 105.86 154.597919) (width 0.25) (layer F.Cu) (net 2))
   (segment (start 115.7 119.4) (end 118 119.4) (width 0.25) (layer F.Cu) (net 3))
-  (via (at 107.6 130.6) (size 0.6) (drill 0.4) (layers F.Cu B.Cu) (net 4))
-  (via (at 109.6 133.2) (size 0.6) (drill 0.4) (layers F.Cu B.Cu) (net 4))
-  (segment (start 104.974999 130.285001) (end 104.974999 128.514999) (width 0.25) (layer F.Cu) (net 4))
-  (segment (start 105.289998 130.6) (end 104.974999 130.285001) (width 0.25) (layer F.Cu) (net 4))
-  (segment (start 107.6 130.6) (end 105.289998 130.6) (width 0.25) (layer F.Cu) (net 4))
-  (segment (start 107.6 131.2) (end 109.6 133.2) (width 0.25) (layer B.Cu) (net 4))
-  (segment (start 107.6 130.6) (end 107.6 131.2) (width 0.25) (layer B.Cu) (net 4))
   (segment (start 111.975 127.6) (end 112.775 126.8) (width 0.25) (layer F.Cu) (net 4))
   (segment (start 111 127.6) (end 111.975 127.6) (width 0.25) (layer F.Cu) (net 4))
   (segment (start 112.775 126.8) (end 113 126.8) (width 0.25) (layer F.Cu) (net 4))
-  (segment (start 112.55 119.4) (end 113.4 119.4) (width 0.25) (layer F.Cu) (net 21))
-  (segment (start 111 120.95) (end 112.55 119.4) (width 0.25) (layer F.Cu) (net 21))
-  (segment (start 111 123.05) (end 111 120.95) (width 0.25) (layer F.Cu) (net 21))
   (segment (start 102.634313 121.505381) (end 99.911953 118.783021) (width 0.25) (layer F.Cu) (net 5))
   (segment (start 106.578942 125.45001) (end 102.634313 121.505381) (width 0.25) (layer F.Cu) (net 5))
@@
   (segment (start 122.4 117.2) (end 125.4 117.2) (width 0.25) (layer B.Cu) (net 14))
   (segment (start 115.4 124.2) (end 122.4 117.2) (width 0.25) (layer B.Cu) (net 14))
+  (segment (start 112.55 119.4) (end 113.4 119.4) (width 0.25) (layer F.Cu) (net 21))
+  (segment (start 111 120.95) (end 112.55 119.4) (width 0.25) (layer F.Cu) (net 21))
+  (segment (start 111 123.05) (end 111 120.95) (width 0.25) (layer F.Cu) (net 21))
   (segment (start 113.4 119.4) (end 113.8 119.4) (width 0.25) (layer F.Cu) (net 21))
   (zone (net 4) (net_name VSS) (layer F.Cu) (hatch edge 0.508)
