File: BusinessCard/Schematics/Card.sch (KiCad schematic (older format))
At the start: 11 parts, among them J1 USB_A, J2 System, J3 ExpansionPort, J4 CapPad1, J5 CapPad2, J6 Programming Port, U1 CH552T

Commit message: Cleaned up card schematics
Parts:
- U1: symbol CH552:CH552T -> Card-rescue:CH552T-CH552
Changed lines of the file:
@@
 $EndDescr
 $Comp
-L CH552:CH552T U1
+L Card-rescue:CH552T-CH552 U1
 U 1 1 5C6D8296
 P 6300 3450
